File: KiCad Circuit Stuff/EEE3088F_MM_Power_Project/EEE3088F_MM_Power_Project.kicad_pcb (KiCad board)
At the start: 2 copper layers, 77.3 x 52.9 mm, 85 parts, among them J1 Conn_01x02, J2 Conn_02x16_Odd_Even, U1 MT3608, U10 DRV8833PWP, U11 SS-12D06-G050, U12 AP22814AW5-7, U14 AP22814AW5-7, U2 INA219AIDCNR, U3 AMS1117-3.3, U4 TPS5430DDAR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

Commit message: finished wiring
Parts:
- moved 9-5V_VSense_TP1 103.3 mm to (163.6, 140.5)
- moved 9V_TP1 72.6 mm to (133.9, 130.0)
- moved 9-5V_R1_TP1 69.6 mm to (164.6, 113.3)
- moved CHRG_VinR_TP1 66.6 mm to (146.3, 124.5)
- moved 3V3_TP1 60.2 mm to (128.0, 102.4)
- moved 9-5V_R2_TP1 55.9 mm to (115.8, 102.4)
- moved CHRG_VinR_TP2 43.3 mm to (160.5, 102.4)
- moved GND_TP1 29.0 mm to (146.1, 104.4)
- moved U14 1.66 mm to (129.4, 138.6)
- moved C32 1.65 mm to (128.1, 135.6)
- moved C28 1.60 mm to (130.7, 135.6)
Routing:
- net /AIN2 (U2): track 0.00 -> 117.9 mm, vias 0 -> 7
- net /AIN1 (U2): track 0.00 -> 107.9 mm, vias 0 -> 10
- net /Battery_Out: track 135.7 -> 167.4 mm, vias 1 -> 3
- net +9V: track 73.9 -> 91.1 mm
- net Net-(C7-Pad1): track 3.63 -> 19.1 mm, vias 0 -> 4
- net Net-(U4-VSENSE): track 2.94 -> 18.3 mm, vias 0 -> 2
- net +3V3: track 96.7 -> 108.1 mm, vias 4 -> 6
- net GND: track 169.5 -> 180.7 mm
- net /Battey_Charger_VDD: track 33.7 -> 41.9 mm
- net +5V: track 116.5 -> 121.7 mm
- net /AOUT2 (U1): track 32.6 -> 34.7 mm
- net /CTRL_EXT_LOAD1: track 8.60 -> 10.3 mm
- net /AOUT1 (U1): track 33.7 -> 35.2 mm
- net /EXT_LOAD1_OUT: track 20.5 -> 22.0 mm

Commit message: Made some final tweaks, and created gerber files
Parts:
- added H1: MountingHole, MountingHole:MountingHole_3.2mm_M3_DIN965_Pad, F.Cu at (139.6, 119.7)
- added H2: MountingHole, MountingHole:MountingHole_3.2mm_M3_DIN965_Pad, F.Cu at (139.6, 99.7)
- added H3: MountingHole, MountingHole:MountingHole_3.2mm_M3_DIN965_Pad, F.Cu at (139.6, 109.7)
- J2: moved to F.Cu
- moved 9-5V_R2_TP1 62.4 mm to (162.9, 143.2)
- moved 9-5V_R1_TP1 22.9 mm to (162.9, 136.1)
- moved CHRG_VinR_TP1 16.4 mm to (159.9, 115.3)
- moved CHRG_VinR_TP2 13.3 mm to (163.6, 115.3)
- moved J2 2.56 mm to (158.6, 146.2), turned to -90 degrees
- moved GND_TP1 1.47 mm to (146.3, 102.9)
- moved 9-5V_VSense_TP1 1.01 mm to (162.9, 139.7)
- moved R12 0.06 mm to (164.5, 132.0)
- moved R14 0.06 mm to (164.5, 129.7)
Connections:
- J2 pad 1: /BOUT2 (U1) -> /BOUT1 (U1)
- J2 pad 10: /BIN2 (U2) -> unconnected-(J2-Pin_10-Pad10)
- J2 pad 11: /EXT_LOAD2_OUT -> unconnected-(J2-Pin_11-Pad11)
- J2 pad 12: unconnected-(J2-Pin_12-Pad12) -> /EXT_LOAD2_OUT
- J2 pad 13: /Fast_Charge_CTRL -> /Battery_Out
- J2 pad 14: /Battery_Out -> /Fast_Charge_CTRL
- J2 pad 15: unconnected-(J2-Pin_15-Pad15) -> /I2C1_SCL
- J2 pad 16: /I2C1_SCL -> unconnected-(J2-Pin_16-Pad16)
- J2 pad 17: /I2C1_SDA -> +3V3
- J2 pad 18: +3V3 -> /I2C1_SDA
- J2 pad 19: GND -> +5V
- J2 pad 2: /BOUT1 (U1) -> /BOUT2 (U1)
- J2 pad 20: +5V -> GND
- J2 pad 21: /EXT_LOAD1_OUT -> +9V
- J2 pad 22: +9V -> /EXT_LOAD1_OUT
- J2 pad 23: GND -> /AIN1 (U2)
- J2 pad 24: /AIN1 (U2) -> GND
- J2 pad 25: /CTRL_EXT_LOAD1 -> /AIN2 (U2)
- J2 pad 26: /AIN2 (U2) -> /CTRL_EXT_LOAD1
- J2 pad 27: /AOUT1 (U2) -> /AIN1 (U1)
- J2 pad 28: /AIN1 (U1) -> /AOUT1 (U2)
- J2 pad 29: /AOUT2 (U2) -> /AIN2 (U1)
- J2 pad 3: /BOUT1 (U2) -> /BIN1 (U1)
- J2 pad 30: /AIN2 (U1) -> /AOUT2 (U2)
- J2 pad 31: /AOUT2 (U1) -> /AOUT1 (U1)
- J2 pad 32: /AOUT1 (U1) -> /AOUT2 (U1)
- J2 pad 4: /BIN1 (U1) -> /BOUT1 (U2)
- J2 pad 5: /BOUT2 (U2) -> /BIN2 (U1)
- J2 pad 6: /BIN2 (U1) -> /BOUT2 (U2)
- J2 pad 7: /CTRL_EXT_LOAD2 -> /BIN1 (U2)
- J2 pad 8: /BIN1 (U2) -> /CTRL_EXT_LOAD2
- J2 pad 9: unconnected-(J2-Pin_9-Pad9) -> /BIN2 (U2)
Routing:
- net /Battey_Charger_VDD: track 41.9 -> 46.9 mm
- net GND: track 180.7 -> 184.9 mm, vias 31 -> 32
- net Net-(C7-Pad1): track 19.1 -> 16.0 mm, vias 4 -> 2
- net /AIN2 (U2): track 117.9 -> 120.3 mm
- net +9V: track 91.1 -> 93.2 mm
- net +5V: track 121.7 -> 123.2 mm
- net +3V3: track 108.1 -> 109.1 mm
- net /Battery_Out: track 167.4 -> 166.9 mm
Other:
- board size 77.3 x 52.9 mm -> 77.3 x 58.5 mm
- board text added: "Joab Kloppers: KLPJOA002 Alex Hillman: HILALE010"

Commit message: added stuff
Other:
- board text added: "Joab Kloppers: KLPJOA002 Alex Hillman: HLLALE010 Group 15"
- board text removed: "Joab Kloppers: KLPJOA002 Alex Hillman: HILALE010"
Changed lines of the file:
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@@
     (property "ki_description" "Generic connector, single row, 01x02, script generated (kicad-library-utils/schlib/autogen/connector/)")
     (property "ki_keywords" "connector")
-    (attr through_hole)
+    (attr through_hole exclude_from_bom)
     (fp_text reference "J1" (at 1 -2.9 90) (layer "F.SilkS")
         (effects (font (size 1 1) (thickness 0.15)))
@@
     (property "ki_description" "Generic connector, double row, 02x16, odd/even pin numbering scheme (row 1 odd numbers, row 2 even numbers), script generated (kicad-library-utils/schlib/autogen/connector/)")
     (property "ki_keywords" "connector")
-    (attr through_hole)
+    (attr through_hole exclude_from_bom)
     (fp_text reference "J2" (at 1.27 -2.33 90) (layer "F.SilkS")
         (effects (font (size 1 1) (thickness 0.15)))
@@
   (gr_rect (start 100 94.4882) (end 177.3 152.95)
     (stroke (width 0.2) (type default)) (fill none) (layer "Edge.Cuts"))
-  (gr_text "Joab Kloppers: KLPJOA002\nAlex Hillman: HILALE010\n" (at 145.9484 99.5172) (layer "F.SilkS")
-    (effects (font (size 1.5 1.5) (thickness 0.3) bold) (justify left bottom))
+  (gr_text "Joab Kloppers: KLPJOA002\nAlex Hillman: HLLALE010\nGroup 15\n" (at 155.956 99.568) (layer "F.SilkS")
+    (effects (font (size 1 1) (thickness 0.2) bold) (justify left bottom))
   )
   (segment (start 137.499863 116.76147) (end 137.46713 116.76147) (width 0.76) (layer "F.Cu") (net 1))

Commit message: Changed JST
Parts:
- J1: footprint Connector_JST:JST_PH_B2B-PH-K_1x02_P2.00mm_Vertical -> Connector_JST:JST_PH_S2B-PH-K_1x02_P2.00mm_Horizontal
- moved J1 2.91 mm to (113.3, 146.2), turned to 0 degrees
Routing:
- net /Battery_In_Before_Switch: track 11.2 -> 9.29 mm
Changed lines of the file:
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@@
       (net 3 "+5V") (pinfunction "1") (pintype "passive"))
   )
-  (footprint "Connector_JST:JST_PH_B2B-PH-K_1x02_P2.00mm_Vertical" (layer "F.Cu")
-    (at 111.25 148.25 -90)
-    (descr "JST PH series connector, B2B-PH-K (http://www.jst-mfg.com/product/pdf/eng/ePH.pdf), generated with kicad-footprint-generator")
-    (tags "connector JST PH side entry")
+  (footprint "Connector_JST:JST_PH_S2B-PH-K_1x02_P2.00mm_Horizontal" (layer "F.Cu")
+    (at 113.2906 146.177)
+    (descr "JST PH series connector, S2B-PH-K (http://www.jst-mfg.com/product/pdf/eng/ePH.pdf), generated with kicad-footprint-generator")
+    (tags "connector JST PH top entry")
     (property "Sheetfile" "EEE3088F_MM_Power_Project.kicad_sch")
     (property "Sheetname" "")
     (property "ki_description" "Generic connector, single row, 01x02, script generated (kicad-library-utils/schlib/autogen/connector/)")
     (property "ki_keywords" "connector")
-    (attr through_hole exclude_from_bom)
-    (fp_text reference "J1" (at 1 -2.9 90) (layer "F.SilkS")
+    (attr through_hole)
+    (fp_text reference "J1" (at 1 -2.55) (layer "F.SilkS")
         (effects (font (size 1 1) (thickness 0.15)))
     )
-    (fp_text value "Conn_01x02" (at 1 4 90) (layer "F.Fab")
+    (fp_text value "Conn_01x02" (at -7.0678 5.588) (layer "F.Fab")
         (effects (font (size 1 1) (thickness 0.15)))
     )
-    (fp_text user "${REFERENCE}" (at 1 1.5 90) (layer "F.Fab")
+    (fp_text user "${REFERENCE}" (at 1 2.5) (layer "F.Fab")
         (effects (font (size 1 1) (thickness 0.15)))
     )
-    (fp_line (start -2.36 -2.11) (end -2.36 -0.86)
+    (fp_line (start -2.06 -1.46) (end -2.06 6.36)
       (stroke (width 0.12) (type solid)) (layer "F.SilkS"))
-    (fp_line (start -2.06 -1.81) (end -2.06 2.91)
+    (fp_line (start -2.06 0.14) (end -1.14 0.14)
       (stroke (width 0.12) (type solid)) (layer "F.SilkS"))
-    (fp_line (start -2.06 -0.5) (end -1.45 -0.5)
+    (fp_line (start -2.06 6.36) (end 4.06 6.36)
       (stroke (width 0.12) (type solid)) (layer "F.SilkS"))
-    (fp_line (start -2.06 0.8) (end -1.45 0.8)
+    (fp_line (start -1.3 2.5) (end -1.3 4.1)
       (stroke (width 0.12) (type solid)) (layer "F.SilkS"))
-    (fp_line (start -2.06 2.91) (end 4.06 2.91)
+    (fp_line (start -1.3 4.1) (end -0.3 4.1)
       (stroke (width 0.12) (type solid)) (layer "F.SilkS"))
-    (fp_line (start -1.45 -1.2) (end -1.45 2.3)
+    (fp_line (start -1.14 -1.46) (end -2.06 -1.46)
       (stroke (width 0.12) (type solid)) (layer "F.SilkS"))
-    (fp_line (start -1.45 2.3) (end 3.45 2.3)
+    (fp_line (start -1.14 0.14) (end -1.14 -1.46)
       (stroke (width 0.12) (type solid)) (layer "F.SilkS"))
-    (fp_line (start -1.11 -2.11) (end -2.36 -2.11)
+    (fp_line (start -0.86 0.14) (end -1.14 0.14)
       (stroke (width 0.12) (type solid)) (layer "F.SilkS"))
-    (fp_line (start -0.6 -2.01) (end -0.6 -1.81)
+    (fp_line (start -0.86 0.14) (end -0.86 -1.075)
       (stroke (width 0.12) (type solid)) (layer "F.SilkS"))
-    (fp_line (start -0.3 -2.01) (end -0.6 -2.01)
+    (fp_line (start -0.8 4.1) (end -0.8 6.36)
       (stroke (width 0.12) (type solid)) (layer "F.SilkS"))
-    (fp_line (start -0.3 -1.91) (end -0.6 -1.91)
+    (fp_line (start -0.3 2.5) (end -1.3 2.5)
       (stroke (width 0.12) (type solid)) (layer "F.SilkS"))
-    (fp_line (start -0.3 -1.81) (end -0.3 -2.01)
+    (fp_line (start -0.3 4.1) (end -0.3 2.5)
       (stroke (width 0.12) (type solid)) (layer "F.SilkS"))
-    (fp_line (start 0.5 -1.81) (end 0.5 -1.2)
+    (fp_line (start -0.3 4.1) (end -0.3 6.36)
       (stroke (width 0.12) (type solid)) (layer "F.SilkS"))
-    (fp_line (start 0.5 -1.2) (end -1.45 -1.2)
+    (fp_line (start 0.5 2) (end 1.5 2)
       (stroke (width 0.12) (type solid)) (layer "F.SilkS"))
-    (fp_line (start 0.9 1.8) (end 1.1 1.8)
+    (fp_line (start 0.5 6.36) (end 0.5 2)
       (stroke (width 0.12) (type solid)) (layer "F.SilkS"))
-    (fp_line (start 0.9 2.3) (end 0.9 1.8)
+    (fp_line (start 1.5 2) (end 1.5 6.36)
       (stroke (width 0.12) (type solid)) (layer "F.SilkS"))
-    (fp_line (start 1 2.3) (end 1 1.8)
+    (fp_line (start 2.3 2.5) (end 3.3 2.5)
       (stroke (width 0.12) (type solid)) (layer "F.SilkS"))
-    (fp_line (start 1.1 1.8) (end 1.1 2.3)
+    (fp_line (start 2.3 4.1) (end 2.3 2.5)
       (stroke (width 0.12) (type solid)) (layer "F.SilkS"))
-    (fp_line (start 1.5 -1.2) (end 1.5 -1.81)
+    (fp_line (start 3.14 -1.46) (end 3.14 0.14)
       (stroke (width 0.12) (type solid)) (layer "F.SilkS"))
-    (fp_line (start 3.45 -1.2) (end 1.5 -1.2)
+    (fp_line (start 3.14 0.14) (end 2.86 0.14)
       (stroke (width 0.12) (type solid)) (layer "F.SilkS"))
-    (fp_line (start 3.45 2.3) (end 3.45 -1.2)
+    (fp_line (start 3.3 2.5) (end 3.3 4.1)
       (stroke (width 0.12) (type solid)) (layer "F.SilkS"))
-    (fp_line (start 4.06 -1.81) (end -2.06 -1.81)
+    (fp_line (start 3.3 4.1) (end 2.3 4.1)
       (stroke (width 0.12) (type solid)) (layer "F.SilkS"))
-    (fp_line (start 4.06 -0.5) (end 3.45 -0.5)
+    (fp_line (start 4.06 -1.46) (end 3.14 -1.46)
       (stroke (width 0.12) (type solid)) (layer "F.SilkS"))
-    (fp_line (start 4.06 0.8) (end 3.45 0.8)
+    (fp_line (start 4.06 0.14) (end 3.14 0.14)
       (stroke (width 0.12) (type solid)) (layer "F.SilkS"))
-    (fp_line (start 4.06 2.91) (end 4.06 -1.81)
+    (fp_line (start 4.06 6.36) (end 4.06 -1.46)
       (stroke (width 0.12) (type solid)) (layer "F.SilkS"))
-    (fp_line (start -2.45 -2.2) (end -2.45 3.3)
+    (fp_line (start -2.45 -1.85) (end -2.45 6.75)
       (stroke (width 0.05) (type solid)) (layer "F.CrtYd"))
-    (fp_line (start -2.45 3.3) (end 4.45 3.3)
+    (fp_line (start -2.45 6.75) (end 4.45 6.75)
       (stroke (width 0.05) (type solid)) (layer "F.CrtYd"))
-    (fp_line (start 4.45 -2.2) (end -2.45 -2.2)
+    (fp_line (start 4.45 -1.85) (end -2.45 -1.85)
       (stroke (width 0.05) (type solid)) (layer "F.CrtYd"))
-    (fp_line (start 4.45 3.3) (end 4.45 -2.2)
+    (fp_line (start 4.45 6.75) (end 4.45 -1.85)
       (stroke (width 0.05) (type solid)) (layer "F.CrtYd"))
-    (fp_line (start -2.36 -2.11) (end -2.36 -0.86)
+    (fp_line (start -1.95 -1.35) (end -1.95 6.25)
+      (stroke (width 0.1) (type solid)) (layer "F.Fab"))
+    (fp_line (start -1.95 6.25) (end 3.95 6.25)
+      (stroke (width 0.1) (type solid)) (layer "F.Fab"))
+    (fp_line (start -1.25 -1.35) (end -1.95 -1.35)
+      (stroke (width 0.1) (type solid)) (layer "F.Fab"))
+    (fp_line (start -1.25 0.25) (end -1.25 -1.35)
       (stroke (width 0.1) (type solid)) (layer "F.Fab"))
-    (fp_line (start -1.95 -1.7) (end -1.95 2.8)
+    (fp_line (start -0.5 1.375) (end 0.5 1.375)
       (stroke (width 0.1) (type solid)) (layer "F.Fab"))
-    (fp_line (start -1.95 2.8) (end 3.95 2.8)
+    (fp_line (start 0 0.875) (end -0.5 1.375)
       (stroke (width 0.1) (type solid)) (layer "F.Fab"))
-    (fp_line (start -1.11 -2.11) (end -2.36 -2.11)
+    (fp_line (start 0.5 1.375) (end 0 0.875)
       (stroke (width 0.1) (type solid)) (layer "F.Fab"))
-    (fp_line (start 3.95 -1.7) (end -1.95 -1.7)
+    (fp_line (start 3.25 -1.35) (end 3.25 0.25)
       (stroke (width 0.1) (type solid)) (layer "F.Fab"))
-    (fp_line (start 3.95 2.8) (end 3.95 -1.7)
+    (fp_line (start 3.25 0.25) (end -1.25 0.25)
       (stroke (width 0.1) (type solid)) (layer "F.Fab"))
-    (pad "1" thru_hole roundrect (at 0 0 270) (size 1.2 1.75) (drill 0.75) (layers "*.Cu" "*.Mask") (roundrect_rratio 0.2083333333)
+    (fp_line (start 3.95 -1.35) (end 3.25 -1.35)
+      (stroke (width 0.1) (type solid)) (layer "F.Fab"))
+    (fp_line (start 3.95 6.25) (end 3.95 -1.35)
+      (stroke (width 0.1) (type solid)) (layer "F.Fab"))
+    (pad "1" thru_hole roundrect (at 0 0) (size 1.2 1.75) (drill 0.75) (layers "*.Cu" "*.Mask") (roundrect_rratio 0.208333)
       (net 68 "/Battery_In_Before_Switch") (pinfunction "Pin_1") (pintype "passive"))
-    (pad "2" thru_hole oval (at 2 0 270) (size 1.2 1.75) (drill 0.75) (layers "*.Cu" "*.Mask")
+    (pad "2" thru_hole oval (at 2 0) (size 1.2 1.75) (drill 0.75) (layers "*.Cu" "*.Mask")
       (net 4 "GND") (pinfunction "Pin_2") (pintype "passive"))
-    (model "${KICAD6_3DMODEL_DIR}/Connector_JST.3dshapes/JST_PH_B2B-PH-K_1x02_P2.00mm_Vertical.wrl"
+    (model "${KICAD6_3DMODEL_DIR}/Connector_JST.3dshapes/JST_PH_S2B-PH-K_1x02_P2.00mm_Horizontal.wrl"
       (offset (xyz 0 0 0))
       (scale (xyz 1 1 1))
@@
     (property "ki_description" "Generic connector, double row, 02x16, odd/even pin numbering scheme (row 1 odd numbers, row 2 even numbers), script generated (kicad-library-utils/schlib/autogen/connector/)")
     (property "ki_keywords" "connector")
-    (attr through_hole exclude_from_bom)
+    (attr through_hole)
     (fp_text reference "J2" (at 1.27 -2.33 90) (layer "F.SilkS")
         (effects (font (size 1 1) (thickness 0.15)))
@@
   (segment (start 155.545025 135.581775) (end 155.8464 135.2804) (width 0.25) (layer "F.Cu") (net 65))
   (segment (start 155.545025 136.793974) (end 155.545025 135.581775) (width 0.25) (layer "F.Cu") (net 65))
-  (segment (start 112.085 147.415) (end 112.085 140.335) (width 1.27) (layer "F.Cu") (net 68))
-  (segment (start 112.085 140.335) (end 110 138.25) (width 1.27) (layer "F.Cu") (net 68))
-  (segment (start 111.25 148.25) (end 112.085 147.415) (width 1.27) (layer "F.Cu") (net 68))
+  (segment (start 113.2906 141.5406) (end 110 138.25) (width 1.27) (layer "F.Cu") (net 68))
+  (segment (start 113.2906 146.177) (end 113.2906 141.5406) (width 1.27) (layer "F.Cu") (net 68))
   (segment (start 112.5115 128.159) (end 111.5615 127.209) (width 0.25) (layer "F.Cu") (net 69))
   (segment (start 110 133.549975) (end 110 127.2955) (width 1.27) (layer "F.Cu") (net 69))
