File: KiCad Circuit Stuff/EEE3088F_MM_Power_Project/EEE3088F_MM_Power_Project.kicad_sch (KiCad schematic)
At the start: 85 parts, among them J1 Conn_02x16_Odd_Even, J2 Conn_01x02, U1 MT3608, U11 SS-12D06-G050, U2 AMS1117-3.3, U3 TP4056, U4 INA219AIDCNR, U4 TYPE-C_16P_QTGM027, U5 HUSB237-AA001-DN06R, U6 TS5A3159DCKR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

Commit message: Made some final tweaks, and created gerber files
Parts:
- added H1, H2, H3: MountingHole, MountingHole:MountingHole_3.2mm_M3_DIN965_Pad, symbol Mechanical:MountingHole_Pad
Connections:
- net +3V3: now also J1.17 (Pin_17); no longer J1.18 (Pin_18)
- net +5V: now also J1.19 (Pin_19); no longer J1.20 (Pin_20)
- net +9V: now also J1.21 (Pin_21); no longer J1.22 (Pin_22)
- net AIN1 (U1): now also J1.27 (Pin_27); no longer J1.28 (Pin_28)
- net AIN1 (U2): now also J1.23 (Pin_23); no longer J1.24 (Pin_24)
- net AIN2 (U1): now also J1.29 (Pin_29); no longer J1.30 (Pin_30)
- net AIN2 (U2): now also J1.25 (Pin_25); no longer J1.26 (Pin_26)
- net AOUT1 (U1): now also J1.31 (Pin_31); no longer J1.32 (Pin_32)
- net AOUT1 (U2): now also J1.28 (Pin_28); no longer J1.27 (Pin_27)
- net AOUT2 (U1): now also J1.32 (Pin_32); no longer J1.31 (Pin_31)
- net AOUT2 (U2): now also J1.30 (Pin_30); no longer J1.29 (Pin_29)
- net BIN1 (U1): now also J1.3 (Pin_3); no longer J1.4 (Pin_4)
- net BIN1 (U2): now also J1.7 (Pin_7); no longer J1.8 (Pin_8)
- net BIN2 (U1): now also J1.5 (Pin_5); no longer J1.6 (Pin_6)
- net BIN2 (U2): now also J1.9 (Pin_9); no longer J1.10 (Pin_10)
- net BOUT1 (U1): now also J1.1 (Pin_1); no longer J1.2 (Pin_2)
- net BOUT1 (U2): now also J1.4 (Pin_4); no longer J1.3 (Pin_3)
- net BOUT2 (U1): now also J1.2 (Pin_2); no longer J1.1 (Pin_1)
- net BOUT2 (U2): now also J1.6 (Pin_6); no longer J1.5 (Pin_5)
- net Battery_Out: now also J1.13 (Pin_13); no longer J1.14 (Pin_14)
- net CTRL_EXT_LOAD1: now also J1.26 (Pin_26); no longer J1.25 (Pin_25)
- net CTRL_EXT_LOAD2: now also J1.8 (Pin_8); no longer J1.7 (Pin_7)
- net EXT_LOAD1_OUT: now also J1.22 (Pin_22); no longer J1.21 (Pin_21)
- net EXT_LOAD2_OUT: now also J1.12 (Pin_12); no longer J1.11 (Pin_11)
- net Fast_Charge_CTRL: now also J1.14 (Pin_14); no longer J1.13 (Pin_13)
- net GND: now also J1.20 (Pin_20), J1.24 (Pin_24), H1.1, H2.1, H3.1; no longer J1.19 (Pin_19), J1.23 (Pin_23)
- net I2C1_SCL: now also J1.15 (Pin_15); no longer J1.16 (Pin_16)
- net I2C1_SDA: now also J1.18 (Pin_18); no longer J1.17 (Pin_17)

Commit message: Changed JST
Parts:
- J2: footprint Connector_JST:JST_PH_B2B-PH-K_1x02_P2.00mm_Vertical -> Connector_JST:JST_PH_S2B-PH-K_1x02_P2.00mm_Horizontal
Changed lines of the file:
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@@
       (effects (font (size 1.27 1.27)) (justify left))
     )
-    (property "Footprint" "Connector_JST:JST_PH_B2B-PH-K_1x02_P2.00mm_Vertical" (at 53.34 118.11 0)
+    (property "Footprint" "Connector_JST:JST_PH_S2B-PH-K_1x02_P2.00mm_Horizontal" (at 53.34 118.11 0)
       (effects (font (size 1.27 1.27)) hide)
     )

Commit message: Added ReadMe and other minor changes
Other:
- moved on the sheet: C11, C12, C6, U7
